Commit message: Shorten name of STL folder

File: 4leggedRobot.urdf (robot description, URDF)
Before this commit: robot materials, 17 links, 16 joints
Links:
- link base_link: geometry collision mesh filename=STL/base_link.stl; visual mesh filename=STL/base_link.stl
- link coxa_BL: geometry visual mesh filename=STL/coxa_bl.stl
- link coxa_BR: geometry visual mesh filename=STL/coxa_br.stl
- link coxa_FL: geometry visual mesh filename=STL/coxa_fl.stl
- link coxa_FR: geometry visual mesh filename=STL/coxa_fr.stl
- link femur_BL: geometry visual mesh filename=STL/femur_bl.stl
- link femur_BR: geometry visual mesh filename=STL/femur_br.stl
- link femur_FL: geometry visual mesh filename=STL/femur_fl.stl
- link femur_FR: geometry visual mesh filename=STL/femur_fr.stl
- link tibia_BL: geometry visual mesh filename=STL/tibia_bl.stl
- link tibia_BR: geometry visual mesh filename=STL/tibia_br.stl
- link tibia_FL: geometry visual mesh filename=STL/tibia_fl.stl
- link tibia_FR: geometry visual mesh filename=STL/tibia_fr.stl
